Commit message: fix urdf file add lidar mesh

File: cad_assembly_amr_final_1/urdf/cad_assembly_amr_final_1.urdf (robot description, URDF)
Before this commit: robot cad_assembly_amr_final_1, 40 links, 39 joints
Links:
- link sensor_laser: geometry collision mesh filename=package://cad_assembly_amr_final_1/meshes/R2000.STL scale=0.001 0.001 0.001; visual mesh filename=package://cad_assembly_amr_final_1/meshes/R2000.STL scale=0.001 0.001 0.001
Joints:
- joint joint_sensor_laser: axis (none) -> 0 0 0; origin xyz=0.18 -0.0325 0.325 rpy=0.0 0.0 0.0 -> xyz=0.18 -0.0325 0.228 rpy=1.57 0 1.57

Commit message: fix lidar coordiate for scan and add odom

File: cad_assembly_amr_final_1/urdf/cad_assembly_amr_final_1.urdf (robot description, URDF)
Before this commit: robot cad_assembly_amr_final_1, 40 links, 39 joints
Joints:
- joint joint_sensor_laser: origin xyz=0.18 -0.0325 0.228 rpy=1.57 0 1.57 -> xyz=0.18 -0.0325 0.228 rpy=0 0 0
