Commit message: fixed odom in real world and tyre contact fix

File: cad_assembly_amr_final_1/urdf/cad_assembly_amr_final_1.xacro (robot description, xacro)
@@ -92,5 +92,5 @@
 <gazebo>
   <plugin filename="libgazebo_ros_control.so" name="control"/>
-  <robotNamespace>/cad_assembly_amr_final_1_controller</robotNamespace>
+  <!-- <robotNamespace>/cad_assembly_amr_final_1_controller</robotNamespace> -->
 </gazebo>
 <gazebo reference="base_link">
@@ -101,11 +101,11 @@
 </gazebo>
 <gazebo reference="right_wheel">
-  <mu1>30000</mu1>
-  <mu2>30000</mu2>
+  <mu1>1000</mu1>
+  <mu2>1000</mu2>
   <selfCollide>true</selfCollide>
 </gazebo>
 <gazebo reference="left_wheel">
-  <mu1>30000</mu1>
-  <mu2>30000</mu2>
+  <mu1>1000</mu1>
+  <mu2>1000</mu2>
   <selfCollide>true</selfCollide>
 </gazebo>
@@ -116,4 +116,9 @@
 </gazebo>
 <!--                     URDF               -->
+ <!-- <link name="world"/> -->
+    <!-- <joint name="fixed" type="floating"> -->
+      <!-- <parent link ="world" /> -->
+      <!-- <child link ="base_link" /> -->
+    <!-- </joint> -->
   <link
     name="base_link">
@@ -201,7 +206,7 @@
     <origin
       xyz="-0.0649400472508853 0.249032118798883 0.0781099999999999"
-      rpy="0 0 0" />
-    <parent
-      link="base_link" />
+      rpy="0 1.56 0" />
+    <parent
+      link="Link35" />
     <child
       link="left_wheel" />
@@ -257,7 +262,7 @@
     <origin
       xyz="-0.0649400472508853 -0.311367881201119 0.0780799999999999"
-      rpy="0 0 0" />
-    <parent
-      link="base_link" />
+      rpy="0 1.56 0" />
+    <parent
+      link="Link34" />
     <child
       link="right_wheel" />

Commit message: remove unwanted files

File: cad_assembly_amr_final_1/urdf/cad_assembly_amr_final_1.xacro (robot description, xacro)
@@ -41,5 +41,5 @@
       <pose>0 0 0 0 0 0</pose>
       <visualize>true</visualize>
-      <update_rate>40</update_rate>
+      <update_rate>100</update_rate>
       <ray>
         <scan>

File: pf_description/urdf/r2000.urdf.xacro (robot description, xacro)
@@ -2,5 +2,5 @@
 <robot xmlns:xacro="http://ros.org/wiki/xacro">
     <xacro:macro name="r2000" params="prefix" >
-        <link name="${prefix}scanner_link" >
+        <link name="${prefix}sensor_laser" >
             <visual>
                 <origin xyz="0 0 0" rpy="1.57 0 1.57" />

File: pf_description/urdf/r2000_world.urdf.xacro (robot description, xacro)
@@ -9,5 +9,5 @@
     <joint name="world_joint" type="fixed">
         <parent link="world" />
-        <child link = "scanner_link" />
+        <child link = "sensor_laser" />
         <origin xyz="0.0 0.0 0.0" rpy="0.0 0.0 0.0" />
     </joint>

File: pf_description/urdf/r2300.urdf.xacro (robot description, xacro)
@@ -2,5 +2,5 @@
 <robot xmlns:xacro="http://ros.org/wiki/xacro">
     <xacro:macro name="r2300" params="prefix" >
-        <link name="${prefix}scanner_link" >
+        <link name="${prefix}sensor_laser" >
             <visual>
                 <origin xyz="-0.00195 0.0158 -0.0094" rpy="-1.57 0 1.57" />

File: pf_description/urdf/r2300_world.urdf.xacro (robot description, xacro)
@@ -9,5 +9,5 @@
     <joint name="world_joint" type="fixed">
         <parent link="world" />
-        <child link = "scanner_link" />
+        <child link = "sensor_laser" />
         <origin xyz="0.0 0.0 0.0" rpy="0.0 0.0 0.0" />
     </joint>

Commit message: add scan merger

File: cad_assembly_amr_final_1/urdf/cad_assembly_amr_final_1.xacro (robot description, xacro)
@@ -6,4 +6,5 @@
   name="cad_assembly_amr_final_1">
 <!-- <include filename="$(find cad_assembly_amr_final_1)/urdf/cad_assembly_amr_final_1.trans" /> -->
+<!-- <include filename="$(find realsense2_description)/urdf/test_d435_multiple_cameras.urdf.xacro" /> -->
 <!--                     GAZEBO_PLUGINS                  -->
   <gazebo>

File: realsense-ros/realsense2_description/urdf/test_d435_multiple_cameras.urdf.xacro (robot description, xacro)
@@ -8,5 +8,5 @@
   </xacro:sensor_d435>
   <xacro:sensor_d435 parent="base_link" name="camera2" use_nominal_extrinsics="$(arg use_nominal_extrinsics)">
-    <origin xyz="-0.1 0 0" rpy="0 0 3.1456"/>
+    <origin xyz="0.18 -0.0325 0.308" rpy="0 0 3.1456"/>
   </xacro:sensor_d435>
 </robot>

Commit message: merge depth scan data with cad model

File: cad_assembly_amr_final_1/urdf/cad_assembly_amr_final_1.xacro (robot description, xacro)
@@ -6,5 +6,4 @@
   name="cad_assembly_amr_final_1">
 <!-- <include filename="$(find cad_assembly_amr_final_1)/urdf/cad_assembly_amr_final_1.trans" /> -->
-<!-- <include filename="$(find realsense2_description)/urdf/test_d435_multiple_cameras.urdf.xacro" /> -->
 <!--                     GAZEBO_PLUGINS                  -->
   <gazebo>

File: realsense-ros/realsense2_description/urdf/test_d435_camera.urdf.xacro (robot description, xacro)
@@ -5,6 +5,5 @@
   <xacro:arg name="use_mesh" default="true" />
   <xacro:include filename="$(find realsense2_description)/urdf/_d435.urdf.xacro" />
-  <link name="base_link" />
-  <xacro:sensor_d435 parent="base_link" use_nominal_extrinsics="$(arg use_nominal_extrinsics)" add_plug="$(arg add_plug)" use_mesh="$(arg use_mesh)">
+  <xacro:sensor_d435 parent="sensor_laser" use_nominal_extrinsics="$(arg use_nominal_extrinsics)" add_plug="$(arg add_plug)" use_mesh="$(arg use_mesh)">
     <origin xyz="0 0 0" rpy="0 0 0"/>
   </xacro:sensor_d435>

Commit message: add bringup.launch fix realsense joint

File: cad_assembly_amr_final_1/urdf/cad_assembly_amr_final_1.xacro (robot description, xacro)
@@ -2197,21 +2197,24 @@
   </joint>
 <!--                     LIDAR LINK               -->
-<link
+  <link
     name="sensor_laser">
     <inertial>
       <origin
-        xyz="0.0 0.0 0.0"
-        rpy="0.0 0.0 0.0" />
-      <mass
-        value="0.01" />
-      <inertia
-        ixx="0.000145833" ixy = "0" ixz ="0"
-               iyy="0.000" iyz = "0"
-               izz="0.000208"  />
-    </inertial>
-    <visual>
-      <origin
-        xyz="0 0 0"
-        rpy="1.56 0 0" />
+        xyz="5.73941775963982E-05 -0.0547817281545586 0.000662361701355196"
+        rpy="0 0 0" />
+      <mass
+        value="1.15411724032787" />
+      <inertia
+        ixx="0.00169670713331925"
+        ixy="8.3068554945323E-08"
+        ixz="-1.47480764218124E-07"
+        iyy="0.00298663361197173"
+        iyz="8.62121560025982E-08"
+        izz="0.00167881991277623" />
+    </inertial>
+    <visual>
+      <origin
+        xyz="0 0 0"
+        rpy="0 0 0" />
       <geometry>
         <mesh
@@ -2227,8 +2230,8 @@
       <origin
         xyz="0 0 0"
-        rpy="1.56 0 0" />
-      <geometry>
-        <mesh
-          filename="package://cad_assembly_amr_final_1/meshes/R2000.STL"  scale="0.001 0.001 0.001" />
+        rpy="0 0 0" />
+      <geometry>
+        <mesh
+          filename="package://cad_assembly_amr_final_1/meshes/R2000.STL" scale="0.001 0.001 0.001" />
       </geometry>
     </collision>
@@ -2245,7 +2248,5 @@
       link="sensor_laser" />
     <axis
-      xyz="0 0 0" />
-  </joint>
-<!-- joint_sensor_laser -->
-    <!-- <origin xyz="0.18 -0.0325 0.325" rpy="0.0 0.0 0.0"/> -->
+      xyz="0 0 0 0 0 0" />
+  </joint>
 </robot>

Commit message: scan segment configure

File: cad_assembly_amr_final_1/urdf/cad_assembly_amr_final_1.xacro (robot description, xacro)
@@ -224,5 +224,5 @@
         rpy="0 0 0" />
       <mass
-        value="1.15411724032787" />
+        value="20.15411724032787" />
       <inertia
         ixx="0.00169670713331966"
@@ -2202,5 +2202,5 @@
       <origin
         xyz="5.73941775963982E-05 -0.0547817281545586 0.000662361701355196"
-        rpy="0 1.57 0" />
+        rpy="0 0 0" />
       <mass
         value="1.15411724032787" />
@@ -2216,4 +2216,18 @@
       <origin
         xyz="0 0 0"
+        rpy="1.57 0 1.57" />
+      <geometry>
+        <mesh
+          filename="package://cad_assembly_amr_final_1/meshes/R2000.STL" scale="0.001 0.001 0.001" />
+      </geometry>
+      <material
+        name="">
+        <color
+          rgba="0.792156862745098 0.819607843137255 0.933333333333333 1" />
+      </material>
+    </visual>
+    <collision>
+      <origin
+        xyz="0 0 0"
         rpy="1.57 3.14 1.57" />
       <geometry>
@@ -2221,18 +2235,4 @@
           filename="package://cad_assembly_amr_final_1/meshes/R2000.STL" scale="0.001 0.001 0.001" />
       </geometry>
-      <material
-        name="">
-        <color
-          rgba="0.792156862745098 0.819607843137255 0.933333333333333 1" />
-      </material>
-    </visual>
-    <collision>
-      <origin
-        xyz="0 0 0"
-        rpy="1.57 3.14 1.57" />
-      <geometry>
-        <mesh
-          filename="package://cad_assembly_amr_final_1/meshes/R2000.STL" scale="0.001 0.001 0.001" />
-      </geometry>
     </collision>
   </link>
@@ -2242,5 +2242,5 @@
     <origin
       xyz="0 0 0"
-      rpy="3.14 0 0" />
+      rpy="0 0 0" />
     <parent
       link="Link15" />

Commit message: urdf edit and fix pcl height

File: cad_assembly_amr_final_1/urdf/cad_assembly_amr_final_1.xacro (robot description, xacro)
@@ -596,4 +596,26 @@
       xyz="0 0 0" />
   </joint>
+<!--  -->
+<link
+    name="depth_camera">
+    <visual>
+      <origin
+        xyz="-0.24 0.03 -0.308"
+        rpy="0 0 0" />
+    </visual>
+  </link>
+  <joint
+    name="depth_camera_joint"
+    type="fixed">
+    <origin
+      xyz="0.26 -0.03 0.158"
+      rpy="0 0 0" />
+    <parent
+      link="base_link" />
+    <child
+      link="depth_camera" />
+    <axis
+      xyz="0 0 0" />
+  </joint>
   <link
     name="Link7">
