Commit message: readded realsense and change parent link

File: realsense-ros/realsense2_description/tests/dual_d415.xacro (robot description, xacro)
@@ -3,9 +3,9 @@
   <xacro:include filename="../urdf/_d415.urdf.xacro" />
   <xacro:arg name="use_nominal_extrinsics" default="True" />
-  <link name="base_link" />
-  <xacro:sensor_d415 parent="base_link" name="camera_bottom">
+  <link name="base_link1" />
+  <xacro:sensor_d415 parent="base_link1" name="camera_bottom">
     <origin xyz="0 0 0" rpy="0 0 0"/>
   </xacro:sensor_d415>
-  <xacro:sensor_d415 parent="base_link" name="camera_top">
+  <xacro:sensor_d415 parent="base_link1" name="camera_top">
     <origin xyz="0 0 0.2" rpy="0 0 0"/>
   </xacro:sensor_d415>

File: realsense-ros/realsense2_description/tests/dual_d435.xacro (robot description, xacro)
@@ -3,9 +3,9 @@
   <xacro:include filename="../urdf/_d435.urdf.xacro" />
   <xacro:arg name="use_nominal_extrinsics" default="True" />
-  <link name="base_link" />
-  <xacro:sensor_d435 parent="base_link" name="camera_bottom">
+  <link name="base_link1" />
+  <xacro:sensor_d435 parent="base_link1" name="camera_bottom">
     <origin xyz="0 0 0" rpy="0 0 0"/>
   </xacro:sensor_d435>
-  <xacro:sensor_d435 parent="base_link" name="camera_top">
+  <xacro:sensor_d435 parent="base_link1" name="camera_top">
     <origin xyz="0 0 0.2" rpy="0 0 0"/>
   </xacro:sensor_d435>

File: realsense-ros/realsense2_description/tests/dual_r410.xacro (robot description, xacro)
@@ -3,9 +3,9 @@
   <xacro:include filename="../urdf/_r410.urdf.xacro" />
   <xacro:arg name="use_nominal_extrinsics" default="True" />
-  <link name="base_link" />
-  <xacro:sensor_r410 parent="base_link" name="camera_bottom" >
+  <link name="base_link1" />
+  <xacro:sensor_r410 parent="base_link1" name="camera_bottom" >
     <origin xyz="0 0 0" rpy="0 0 0"/>
   </xacro:sensor_r410>
-  <xacro:sensor_r410 parent="base_link" name="camera_top">
+  <xacro:sensor_r410 parent="base_link1" name="camera_top">
     <origin xyz="0 0 0.2" rpy="0 0 0"/>
   </xacro:sensor_r410>

File: realsense-ros/realsense2_description/tests/dual_r430.xacro (robot description, xacro)
@@ -3,9 +3,9 @@
   <xacro:include filename="../urdf/_r430.urdf.xacro" />
   <xacro:arg name="use_nominal_extrinsics" default="True" />
-  <link name="base_link" />
-  <xacro:sensor_r430 parent="base_link" name="camera_bottom">
+  <link name="base_link1" />
+  <xacro:sensor_r430 parent="base_link1" name="camera_bottom">
     <origin xyz="0 0 0" rpy="0 0 0"/>
   </xacro:sensor_r430>
-  <xacro:sensor_r430 parent="base_link" name="camera_top">
+  <xacro:sensor_r430 parent="base_link1" name="camera_top">
     <origin xyz="0 0 0.2" rpy="0 0 0"/>
   </xacro:sensor_r430>

File: realsense-ros/realsense2_description/tests/one_of_each.xacro (robot description, xacro)
@@ -6,15 +6,15 @@
   <xacro:include filename="../urdf/_r430.urdf.xacro" />
   <xacro:arg name="use_nominal_extrinsics" default="True" />
-  <link name="base_link" />
-  <xacro:sensor_d415 parent="base_link" name="d415">
+  <link name="base_link1" />
+  <xacro:sensor_d415 parent="base_link1" name="d415">
     <origin xyz="0 0 0" rpy="0 0 0"/>
   </xacro:sensor_d415>
-  <xacro:sensor_d435 parent="base_link" name="d435">
+  <xacro:sensor_d435 parent="base_link1" name="d435">
     <origin xyz="0 0 0.1" rpy="0 0 0"/>
   </xacro:sensor_d435>
-  <xacro:sensor_r410 parent="base_link" name="r410">
+  <xacro:sensor_r410 parent="base_link1" name="r410">
     <origin xyz="0 0 0.2" rpy="0 0 0"/>
   </xacro:sensor_r410>
-  <xacro:sensor_r430 parent="base_link" name="r430">
+  <xacro:sensor_r430 parent="base_link1" name="r430">
     <origin xyz="0 0 0.3" rpy="0 0 0"/>
   </xacro:sensor_r430>

File: realsense-ros/realsense2_description/urdf/test_d415_camera.urdf.xacro (robot description, xacro)
@@ -5,6 +5,6 @@
   <xacro:arg name="use_mesh" default="true" />
   <xacro:include filename="$(find realsense2_description)/urdf/_d415.urdf.xacro" />
-  <link name="base_link" />
-  <xacro:sensor_d415 parent="base_link" use_nominal_extrinsics="$(arg use_nominal_extrinsics)" add_plug="$(arg add_plug)" use_mesh="$(arg use_mesh)">
+  <link name="base_link1" />
+  <xacro:sensor_d415 parent="base_link1" use_nominal_extrinsics="$(arg use_nominal_extrinsics)" add_plug="$(arg add_plug)" use_mesh="$(arg use_mesh)">
     <origin xyz="0 0 0" rpy="0 0 0"/>
   </xacro:sensor_d415>

File: realsense-ros/realsense2_description/urdf/test_d435_camera.urdf.xacro (robot description, xacro)
@@ -5,5 +5,6 @@
   <xacro:arg name="use_mesh" default="true" />
   <xacro:include filename="$(find realsense2_description)/urdf/_d435.urdf.xacro" />
-  <xacro:sensor_d435 parent="sensor_laser" use_nominal_extrinsics="$(arg use_nominal_extrinsics)" add_plug="$(arg add_plug)" use_mesh="$(arg use_mesh)">
+  <link name="base_link1" />
+  <xacro:sensor_d435 parent="base_link1" use_nominal_extrinsics="$(arg use_nominal_extrinsics)" add_plug="$(arg add_plug)" use_mesh="$(arg use_mesh)">
     <origin xyz="0 0 0" rpy="0 0 0"/>
   </xacro:sensor_d435>

File: realsense-ros/realsense2_description/urdf/test_d435_multiple_cameras.urdf.xacro (robot description, xacro)
@@ -3,10 +3,10 @@
   <xacro:arg name="use_nominal_extrinsics" default="false"/>
   <xacro:include filename="$(find realsense2_description)/urdf/_d435.urdf.xacro" />
-  <link name="base_link" />
-  <xacro:sensor_d435 parent="base_link" name="camera1" use_nominal_extrinsics="$(arg use_nominal_extrinsics)">
+  <link name="base_link1" />
+  <xacro:sensor_d435 parent="base_link1" name="camera1" use_nominal_extrinsics="$(arg use_nominal_extrinsics)">
     <origin xyz="0.1 0 0" rpy="0 0 0"/>
   </xacro:sensor_d435>
-  <xacro:sensor_d435 parent="base_link" name="camera2" use_nominal_extrinsics="$(arg use_nominal_extrinsics)">
-    <origin xyz="0.18 -0.0325 0.308" rpy="0 0 3.1456"/>
+  <xacro:sensor_d435 parent="base_link1" name="camera2" use_nominal_extrinsics="$(arg use_nominal_extrinsics)">
+    <origin xyz="-0.1 0 0" rpy="0 0 3.1456"/>
   </xacro:sensor_d435>
 </robot>

File: realsense-ros/realsense2_description/urdf/test_d435i_camera.urdf.xacro (robot description, xacro)
@@ -3,6 +3,6 @@
   <xacro:arg name="use_nominal_extrinsics" default="false" />
   <xacro:include filename="$(find realsense2_description)/urdf/_d435i.urdf.xacro"/>
-  <link name="base_link" />
-  <xacro:sensor_d435i parent="base_link" use_nominal_extrinsics="$(arg use_nominal_extrinsics)">
+  <link name="base_link1" />
+  <xacro:sensor_d435i parent="base_link1" use_nominal_extrinsics="$(arg use_nominal_extrinsics)">
     <origin xyz="0 0 0" rpy="0 0 0"/>
   </xacro:sensor_d435i>

File: realsense-ros/realsense2_description/urdf/test_d455_camera.urdf.xacro (robot description, xacro)
@@ -3,6 +3,6 @@
   <xacro:arg name="use_nominal_extrinsics" default="false"/>
   <xacro:include filename="$(find realsense2_description)/urdf/_d455.urdf.xacro" />
-  <link name="base_link" />
-  <xacro:sensor_d455 parent="base_link" use_nominal_extrinsics="$(arg use_nominal_extrinsics)">
+  <link name="base_link1" />
+  <xacro:sensor_d455 parent="base_link1" use_nominal_extrinsics="$(arg use_nominal_extrinsics)">
     <origin xyz="0 0 0" rpy="0 0 0"/>
   </xacro:sensor_d455>

File: realsense-ros/realsense2_description/urdf/test_l515_camera.urdf.xacro (robot description, xacro)
@@ -5,6 +5,6 @@
   <xacro:arg name="use_mesh" default="true" />
   <xacro:include filename="$(find realsense2_description)/urdf/_l515.urdf.xacro" />
-  <link name="base_link" />
-  <xacro:sensor_l515 parent="base_link" use_nominal_extrinsics="$(arg use_nominal_extrinsics)" add_plug="$(arg add_plug)" use_mesh="$(arg use_mesh)">
+  <link name="base_link1" />
+  <xacro:sensor_l515 parent="base_link1" use_nominal_extrinsics="$(arg use_nominal_extrinsics)" add_plug="$(arg add_plug)" use_mesh="$(arg use_mesh)">
     <origin xyz="0 0 0" rpy="0 0 0"/>
   </xacro:sensor_l515>

File: realsense-ros/realsense2_description/urdf/test_r410_camera.urdf.xacro (robot description, xacro)
@@ -3,6 +3,6 @@
   <xacro:arg name="use_nominal_extrinsics" default="false"/>
   <xacro:include filename="$(find realsense2_description)/urdf/_r410.urdf.xacro" />
-  <link name="base_link" />
-  <xacro:sensor_r410 parent="base_link" use_nominal_extrinsics="$(arg use_nominal_extrinsics)">
+  <link name="base_link1" />
+  <xacro:sensor_r410 parent="base_link1" use_nominal_extrinsics="$(arg use_nominal_extrinsics)">
     <origin xyz="0 0 0" rpy="0 0 0"/>
   </xacro:sensor_r410>

File: realsense-ros/realsense2_description/urdf/test_r430_camera.urdf.xacro (robot description, xacro)
@@ -3,6 +3,6 @@
   <xacro:arg name="use_nominal_extrinsics" default="false"/>
   <xacro:include filename="$(find realsense2_description)/urdf/_r430.urdf.xacro" />
-  <link name="base_link" />
-  <xacro:sensor_r430 parent="base_link" use_nominal_extrinsics="$(arg use_nominal_extrinsics)">
+  <link name="base_link1" />
+  <xacro:sensor_r430 parent="base_link1" use_nominal_extrinsics="$(arg use_nominal_extrinsics)">
     <origin xyz="0 0 0" rpy="0 0 0"/>
   </xacro:sensor_r430>

Commit message: added passthrough filter in point cloud

File: realsense-ros/realsense2_description/tests/dual_d415.xacro (robot description, xacro)
@@ -3,9 +3,9 @@
   <xacro:include filename="../urdf/_d415.urdf.xacro" />
   <xacro:arg name="use_nominal_extrinsics" default="True" />
-  <link name="base_link1" />
-  <xacro:sensor_d415 parent="base_link1" name="camera_bottom">
+  <link name="base_link" />
+  <xacro:sensor_d415 parent="base_link" name="camera_bottom">
     <origin xyz="0 0 0" rpy="0 0 0"/>
   </xacro:sensor_d415>
-  <xacro:sensor_d415 parent="base_link1" name="camera_top">
+  <xacro:sensor_d415 parent="base_link" name="camera_top">
     <origin xyz="0 0 0.2" rpy="0 0 0"/>
   </xacro:sensor_d415>

File: realsense-ros/realsense2_description/tests/dual_d435.xacro (robot description, xacro)
@@ -3,9 +3,9 @@
   <xacro:include filename="../urdf/_d435.urdf.xacro" />
   <xacro:arg name="use_nominal_extrinsics" default="True" />
-  <link name="base_link1" />
-  <xacro:sensor_d435 parent="base_link1" name="camera_bottom">
+  <link name="base_link" />
+  <xacro:sensor_d435 parent="base_link" name="camera_bottom">
     <origin xyz="0 0 0" rpy="0 0 0"/>
   </xacro:sensor_d435>
-  <xacro:sensor_d435 parent="base_link1" name="camera_top">
+  <xacro:sensor_d435 parent="base_link" name="camera_top">
     <origin xyz="0 0 0.2" rpy="0 0 0"/>
   </xacro:sensor_d435>

File: realsense-ros/realsense2_description/tests/dual_r410.xacro (robot description, xacro)
@@ -3,9 +3,9 @@
   <xacro:include filename="../urdf/_r410.urdf.xacro" />
   <xacro:arg name="use_nominal_extrinsics" default="True" />
-  <link name="base_link1" />
-  <xacro:sensor_r410 parent="base_link1" name="camera_bottom" >
+  <link name="base_link" />
+  <xacro:sensor_r410 parent="base_link" name="camera_bottom" >
     <origin xyz="0 0 0" rpy="0 0 0"/>
   </xacro:sensor_r410>
-  <xacro:sensor_r410 parent="base_link1" name="camera_top">
+  <xacro:sensor_r410 parent="base_link" name="camera_top">
     <origin xyz="0 0 0.2" rpy="0 0 0"/>
   </xacro:sensor_r410>

File: realsense-ros/realsense2_description/tests/dual_r430.xacro (robot description, xacro)
@@ -3,9 +3,9 @@
   <xacro:include filename="../urdf/_r430.urdf.xacro" />
   <xacro:arg name="use_nominal_extrinsics" default="True" />
-  <link name="base_link1" />
-  <xacro:sensor_r430 parent="base_link1" name="camera_bottom">
+  <link name="base_link" />
+  <xacro:sensor_r430 parent="base_link" name="camera_bottom">
     <origin xyz="0 0 0" rpy="0 0 0"/>
   </xacro:sensor_r430>
-  <xacro:sensor_r430 parent="base_link1" name="camera_top">
+  <xacro:sensor_r430 parent="base_link" name="camera_top">
     <origin xyz="0 0 0.2" rpy="0 0 0"/>
   </xacro:sensor_r430>

File: realsense-ros/realsense2_description/tests/one_of_each.xacro (robot description, xacro)
@@ -6,15 +6,15 @@
   <xacro:include filename="../urdf/_r430.urdf.xacro" />
   <xacro:arg name="use_nominal_extrinsics" default="True" />
-  <link name="base_link1" />
-  <xacro:sensor_d415 parent="base_link1" name="d415">
+  <link name="base_link" />
+  <xacro:sensor_d415 parent="base_link" name="d415">
     <origin xyz="0 0 0" rpy="0 0 0"/>
   </xacro:sensor_d415>
-  <xacro:sensor_d435 parent="base_link1" name="d435">
+  <xacro:sensor_d435 parent="base_link" name="d435">
     <origin xyz="0 0 0.1" rpy="0 0 0"/>
   </xacro:sensor_d435>
-  <xacro:sensor_r410 parent="base_link1" name="r410">
+  <xacro:sensor_r410 parent="base_link" name="r410">
     <origin xyz="0 0 0.2" rpy="0 0 0"/>
   </xacro:sensor_r410>
-  <xacro:sensor_r430 parent="base_link1" name="r430">
+  <xacro:sensor_r430 parent="base_link" name="r430">
     <origin xyz="0 0 0.3" rpy="0 0 0"/>
   </xacro:sensor_r430>

File: realsense-ros/realsense2_description/urdf/test_d415_camera.urdf.xacro (robot description, xacro)
@@ -5,6 +5,6 @@
   <xacro:arg name="use_mesh" default="true" />
   <xacro:include filename="$(find realsense2_description)/urdf/_d415.urdf.xacro" />
-  <link name="base_link1" />
-  <xacro:sensor_d415 parent="base_link1" use_nominal_extrinsics="$(arg use_nominal_extrinsics)" add_plug="$(arg add_plug)" use_mesh="$(arg use_mesh)">
+  <link name="base_link" />
+  <xacro:sensor_d415 parent="base_link" use_nominal_extrinsics="$(arg use_nominal_extrinsics)" add_plug="$(arg add_plug)" use_mesh="$(arg use_mesh)">
     <origin xyz="0 0 0" rpy="0 0 0"/>
   </xacro:sensor_d415>

File: realsense-ros/realsense2_description/urdf/test_d435_camera.urdf.xacro (robot description, xacro)
@@ -5,6 +5,6 @@
   <xacro:arg name="use_mesh" default="true" />
   <xacro:include filename="$(find realsense2_description)/urdf/_d435.urdf.xacro" />
-  <link name="base_link1" />
-  <xacro:sensor_d435 parent="base_link1" use_nominal_extrinsics="$(arg use_nominal_extrinsics)" add_plug="$(arg add_plug)" use_mesh="$(arg use_mesh)">
+  <link name="base_link" />
+  <xacro:sensor_d435 parent="base_link" use_nominal_extrinsics="$(arg use_nominal_extrinsics)" add_plug="$(arg add_plug)" use_mesh="$(arg use_mesh)">
     <origin xyz="0 0 0" rpy="0 0 0"/>
   </xacro:sensor_d435>

File: realsense-ros/realsense2_description/urdf/test_d435_multiple_cameras.urdf.xacro (robot description, xacro)
@@ -3,9 +3,9 @@
   <xacro:arg name="use_nominal_extrinsics" default="false"/>
   <xacro:include filename="$(find realsense2_description)/urdf/_d435.urdf.xacro" />
-  <link name="base_link1" />
-  <xacro:sensor_d435 parent="base_link1" name="camera1" use_nominal_extrinsics="$(arg use_nominal_extrinsics)">
+  <link name="base_link" />
+  <xacro:sensor_d435 parent="base_link" name="camera1" use_nominal_extrinsics="$(arg use_nominal_extrinsics)">
     <origin xyz="0.1 0 0" rpy="0 0 0"/>
   </xacro:sensor_d435>
-  <xacro:sensor_d435 parent="base_link1" name="camera2" use_nominal_extrinsics="$(arg use_nominal_extrinsics)">
+  <xacro:sensor_d435 parent="base_link" name="camera2" use_nominal_extrinsics="$(arg use_nominal_extrinsics)">
     <origin xyz="-0.1 0 0" rpy="0 0 3.1456"/>
   </xacro:sensor_d435>

File: realsense-ros/realsense2_description/urdf/test_d435i_camera.urdf.xacro (robot description, xacro)
@@ -3,6 +3,6 @@
   <xacro:arg name="use_nominal_extrinsics" default="false" />
   <xacro:include filename="$(find realsense2_description)/urdf/_d435i.urdf.xacro"/>
-  <link name="base_link1" />
-  <xacro:sensor_d435i parent="base_link1" use_nominal_extrinsics="$(arg use_nominal_extrinsics)">
+  <link name="base_link" />
+  <xacro:sensor_d435i parent="base_link" use_nominal_extrinsics="$(arg use_nominal_extrinsics)">
     <origin xyz="0 0 0" rpy="0 0 0"/>
   </xacro:sensor_d435i>

File: realsense-ros/realsense2_description/urdf/test_d455_camera.urdf.xacro (robot description, xacro)
@@ -3,6 +3,6 @@
   <xacro:arg name="use_nominal_extrinsics" default="false"/>
   <xacro:include filename="$(find realsense2_description)/urdf/_d455.urdf.xacro" />
-  <link name="base_link1" />
-  <xacro:sensor_d455 parent="base_link1" use_nominal_extrinsics="$(arg use_nominal_extrinsics)">
+  <link name="base_link" />
+  <xacro:sensor_d455 parent="base_link" use_nominal_extrinsics="$(arg use_nominal_extrinsics)">
     <origin xyz="0 0 0" rpy="0 0 0"/>
   </xacro:sensor_d455>

File: realsense-ros/realsense2_description/urdf/test_l515_camera.urdf.xacro (robot description, xacro)
@@ -5,6 +5,6 @@
   <xacro:arg name="use_mesh" default="true" />
   <xacro:include filename="$(find realsense2_description)/urdf/_l515.urdf.xacro" />
-  <link name="base_link1" />
-  <xacro:sensor_l515 parent="base_link1" use_nominal_extrinsics="$(arg use_nominal_extrinsics)" add_plug="$(arg add_plug)" use_mesh="$(arg use_mesh)">
+  <link name="base_link" />
+  <xacro:sensor_l515 parent="base_link" use_nominal_extrinsics="$(arg use_nominal_extrinsics)" add_plug="$(arg add_plug)" use_mesh="$(arg use_mesh)">
     <origin xyz="0 0 0" rpy="0 0 0"/>
   </xacro:sensor_l515>

File: realsense-ros/realsense2_description/urdf/test_r410_camera.urdf.xacro (robot description, xacro)
@@ -3,6 +3,6 @@
   <xacro:arg name="use_nominal_extrinsics" default="false"/>
   <xacro:include filename="$(find realsense2_description)/urdf/_r410.urdf.xacro" />
-  <link name="base_link1" />
-  <xacro:sensor_r410 parent="base_link1" use_nominal_extrinsics="$(arg use_nominal_extrinsics)">
+  <link name="base_link" />
+  <xacro:sensor_r410 parent="base_link" use_nominal_extrinsics="$(arg use_nominal_extrinsics)">
     <origin xyz="0 0 0" rpy="0 0 0"/>
   </xacro:sensor_r410>

File: realsense-ros/realsense2_description/urdf/test_r430_camera.urdf.xacro (robot description, xacro)
@@ -3,6 +3,6 @@
   <xacro:arg name="use_nominal_extrinsics" default="false"/>
   <xacro:include filename="$(find realsense2_description)/urdf/_r430.urdf.xacro" />
-  <link name="base_link1" />
-  <xacro:sensor_r430 parent="base_link1" use_nominal_extrinsics="$(arg use_nominal_extrinsics)">
+  <link name="base_link" />
+  <xacro:sensor_r430 parent="base_link" use_nominal_extrinsics="$(arg use_nominal_extrinsics)">
     <origin xyz="0 0 0" rpy="0 0 0"/>
   </xacro:sensor_r430>
